File: das48-ESP32/untitled.brd (EAGLE design)
At the start: 271.6 x 104.1 mm, 431 parts, among them IC1 MCP23017SS, IC4 MCP23017SS, IC5 MCP23017SS, J3 10118193-0001LF, K1 SRD-05VDC-SL-C, Q1 S9013, Q2 MMBT3904, Q3 MMBT3904, Q4 12MHz, Q5 S9013, Q6 S9013, Q7 S9013, Q8 S9013, U1 CH340G, U2 AMS1117, U3 ESP32-WROOM-32D, U4 PC817X2NIP0F, U49 PC817X2NIP0F, U5 PC817X2NIP0F, U6 PC817X2NIP0F, U7 PC817X2NIP0F, X1 22-23-2031

Commit message: revisi tanggal 09/02/2023(revisi mas naufal)
Parts:
- added D107: US1M-13, US1M-13:DIOM5226X240N
- added JP1: (no value), pinhead:1X04
- added K2: 351, relay:351
- added Q9: S9013, S9013:SOT95P240X120-3N
- added R138: 330, adafruit:M0805
- added R139: 10k, adafruit:M0805
- added RTC1: (no value), rtc3231:RTC3231
- added U8: PC817X2NIP0F, PC817X2NIP0F:SOT254P975X400-4N
- moved R130 65.6 mm to (-8.55, 102.2)
- moved D103 65.6 mm to (-6.18, 102.2)
- moved R129 65.5 mm to (-3.92, 102.2)
- moved D51 65.5 mm to (0.98, 66.0)
- moved TTL-RS1 65.4 mm to (36.5, 89.1)
- moved R4 65.2 mm to (45.1, 125.6), flipped to the top
- moved S1 65.0 mm to (-37.6, 130.0), flipped to the top, turned to 270 degrees
- moved D11 65.0 mm to (86.5, 124.3)
- moved D13 65.0 mm to (100.7, 124.2)
- moved D15 65.0 mm to (114.9, 124.2)
- moved D41 65.0 mm to (121.0, 69.7)
- moved D64 65.0 mm to (89.1, 124.3)
- moved D89 65.0 mm to (82.9, 69.8)
- moved D93 65.0 mm to (111.4, 69.7)
- moved LED13 65.0 mm to (112.7, 113.9)
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Connections:
- new net COMM1: K2.P1, OPTO1.2, OPTO10.2, OPTO11.2, OPTO12.2, OPTO13.2, OPTO14.2, OPTO15.2, OPTO16.2, OPTO17.2, OPTO18.2, OPTO19.2, OPTO2.2, OPTO20.2, OPTO21.2, OPTO22.2, OPTO23.2, OPTO24.2, OPTO25.2, OPTO26.2, OPTO27.2, OPTO28.2, OPTO29.2, OPTO3.2, OPTO30.2, OPTO31.2, OPTO32.2, OPTO33.2, OPTO34.2, OPTO35.2, OPTO36.2, OPTO37.2, OPTO38.2, OPTO39.2, OPTO4.2, OPTO40.2, OPTO41.2, OPTO42.2, OPTO43.2, OPTO44.2, OPTO45.2, OPTO46.2, OPTO47.2, OPTO48.2, OPTO5.2, OPTO6.2, OPTO7.2, OPTO8.2, OPTO9.2, Z1.A, Z10.A, Z11.A, Z12.A, Z13.A, Z14.A, Z15.A, Z16.A, Z17.A, Z18.A, Z19.A, Z2.A, Z20.A, Z21.A, Z22.A, Z23.A, Z24.A, Z25.A, Z26.A, Z27.A, Z28.A, Z29.A, Z3.A, Z30.A, Z31.A, Z32.A, Z33.A, Z34.A, Z35.A, Z36.A, Z37.A, Z38.A, Z39.A, Z4.A, Z40.A, Z41.A, Z42.A, Z43.A, Z44.A, Z45.A, Z46.A, Z47.A, Z48.A, Z5.A, Z6.A, Z7.A, Z8.A, Z9.A
- new net GND_TEST: R138.1, U3.12
- new net N$54: R138.2, U8.1
- new net N$58: R139.1, U8.4
- new net N$62: Q9.1, U8.3
- new net N$73: D107.A, K2.16, Q9.3
- new net RX_BACKUP: JP1.2, U3.9
- new net TX_BACKUP: JP1.3, U3.8
- net COMM: now also K2.O1; no longer OPTO1.2, OPTO10.2, OPTO11.2, OPTO12.2, OPTO13.2, OPTO14.2, OPTO15.2, OPTO16.2, OPTO17.2, OPTO18.2, OPTO19.2, OPTO2.2, OPTO20.2, OPTO21.2, OPTO22.2, OPTO23.2, OPTO24.2, OPTO25.2, OPTO26.2, OPTO27.2, OPTO28.2, OPTO29.2, OPTO3.2, OPTO30.2, OPTO31.2, OPTO32.2, OPTO33.2, OPTO34.2, OPTO35.2, OPTO36.2, OPTO37.2, OPTO38.2, OPTO39.2, OPTO4.2, OPTO40.2, OPTO41.2, OPTO42.2, OPTO43.2, OPTO44.2, OPTO45.2, OPTO46.2, OPTO47.2, OPTO48.2, OPTO5.2, OPTO6.2, OPTO7.2, OPTO8.2, OPTO9.2, Z1.A, Z10.A, Z11.A, Z12.A, Z13.A, Z14.A, Z15.A, Z16.A, Z17.A, Z18.A, Z19.A, Z2.A, Z20.A, Z21.A, Z22.A, Z23.A, Z24.A, Z25.A, Z26.A, Z27.A, Z28.A, Z29.A, Z3.A, Z30.A, Z31.A, Z32.A, Z33.A, Z34.A, Z35.A, Z36.A, Z37.A, Z38.A, Z39.A, Z4.A, Z40.A, Z41.A, Z42.A, Z43.A, Z44.A, Z45.A, Z46.A, Z47.A, Z48.A, Z5.A, Z6.A, Z7.A, Z8.A, Z9.A
- net GND: now also JP1.4, K2.S1, Q9.2, RTC1.GND, U8.2
- net LED_PROSES: now also U3.10
- net LED_WARNING: now also U3.11
- net OUT+: now also D107.C, JP1.1, K2.1, R139.2
- net SCL: now also RTC1.SCL
- net SDA: now also RTC1.SDA
- net VCC: now also RTC1.VCC
Routing:
- net COMM1: track 0.00 -> 1444.7 mm, vias 0 -> 2
- net COMM: track 1132.4 -> 295.4 mm, vias 2 -> 0
- net GND: track 1095.8 -> 1258.6 mm, vias 26 -> 31
- net SCL: track 373.9 -> 490.1 mm
- net LED_PROSES: track 0.00 -> 69.3 mm, vias 0 -> 2
- net LED_WARNING: track 0.00 -> 66.4 mm, vias 0 -> 2
- net SDA: track 314.6 -> 379.7 mm
- net VCC: track 943.2 -> 1001.0 mm
- net OUT+: track 304.7 -> 351.3 mm, vias 6 -> 8
- net N$62: track 0.00 -> 43.7 mm, vias 0 -> 3
- net RX_BACKUP: track 0.00 -> 33.9 mm, vias 0 -> 1
- net TX_BACKUP: track 0.00 -> 33.6 mm, vias 0 -> 1
- net GND_TEST: track 0.00 -> 24.9 mm, vias 0 -> 1
- net N$54: track 0.00 -> 20.1 mm, vias 0 -> 1
- net N$58: track 0.00 -> 12.8 mm, vias 0 -> 1
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Other:
- outline, holes or cut-outs redrawn
