File: das48-ESP32/untitled.sch (EAGLE design)
At the start: 431 parts, among them IC1 MCP23017SS, IC4 MCP23017SS, IC5 MCP23017SS, J3 10118193-0001LF, K1 SRD-05VDC-SL-C, Q1 S9013, Q2 MMBT3904, Q3 MMBT3904, Q4 12MHz, Q5 S9013, Q6 S9013, Q7 S9013, Q8 S9013, U1 CH340G, U2 AMS1117, U3 ESP32-WROOM-32D, U4 PC817X2NIP0F, U49 PC817X2NIP0F, U5 PC817X2NIP0F, U6 PC817X2NIP0F, U7 PC817X2NIP0F, X1 22-23-2031

Commit message: revisi tanggal 09/02/2023(revisi mas naufal)
Parts:
- added D107: US1M-13, US1M-13:US1M-13
- added JP1: (no value), pinhead:PINHD-1X4
- added K2: 351, relay:351
- added Q9: S9013, S9013:S9013
- added R138: 330, adafruit:R-US_M0805
- added R139: 10k, adafruit:R-US_M0805
- added RTC1: (no value), rtc3231:RTC3231
- added U8: PC817X2NIP0F, PC817X2NIP0F:PC817X2NIP0F
Connections:
- new net COMM1: K22.P, OPTO1.C, OPTO10.C, OPTO11.C, OPTO12.C, OPTO13.C, OPTO14.C, OPTO15.C, OPTO16.C, OPTO17.C, OPTO18.C, OPTO19.C, OPTO2.C, OPTO20.C, OPTO21.C, OPTO22.C, OPTO23.C, OPTO24.C, OPTO25.C, OPTO26.C, OPTO27.C, OPTO28.C, OPTO29.C, OPTO3.C, OPTO30.C, OPTO31.C, OPTO32.C, OPTO33.C, OPTO34.C, OPTO35.C, OPTO36.C, OPTO37.C, OPTO38.C, OPTO39.C, OPTO4.C, OPTO40.C, OPTO41.C, OPTO42.C, OPTO43.C, OPTO44.C, OPTO45.C, OPTO46.C, OPTO47.C, OPTO48.C, OPTO5.C, OPTO6.C, OPTO7.C, OPTO8.C, OPTO9.C, Z1.A, Z10.A, Z11.A, Z12.A, Z13.A, Z14.A, Z15.A, Z16.A, Z17.A, Z18.A, Z19.A, Z2.A, Z20.A, Z21.A, Z22.A, Z23.A, Z24.A, Z25.A, Z26.A, Z27.A, Z28.A, Z29.A, Z3.A, Z30.A, Z31.A, Z32.A, Z33.A, Z34.A, Z35.A, Z36.A, Z37.A, Z38.A, Z39.A, Z4.A, Z40.A, Z41.A, Z42.A, Z43.A, Z44.A, Z45.A, Z46.A, Z47.A, Z48.A, Z5.A, Z6.A, Z7.A, Z8.A, Z9.A
- new net GND_TEST: R138.1, U3.IO27
- new net N$54: R138.2, U8.A
- new net N$58: R139.1, U8.CT
- new net N$62: Q9.B, U8.ET
- new net N$73: D107.A, K21.2, Q9.C
- new net RX_BACKUP: JP1.2, U3.IO33
- new net TX_BACKUP: JP1.3, U3.IO32
- net COMM: now also K22.O; no longer OPTO1.C, OPTO10.C, OPTO11.C, OPTO12.C, OPTO13.C, OPTO14.C, OPTO15.C, OPTO16.C, OPTO17.C, OPTO18.C, OPTO19.C, OPTO2.C, OPTO20.C, OPTO21.C, OPTO22.C, OPTO23.C, OPTO24.C, OPTO25.C, OPTO26.C, OPTO27.C, OPTO28.C, OPTO29.C, OPTO3.C, OPTO30.C, OPTO31.C, OPTO32.C, OPTO33.C, OPTO34.C, OPTO35.C, OPTO36.C, OPTO37.C, OPTO38.C, OPTO39.C, OPTO4.C, OPTO40.C, OPTO41.C, OPTO42.C, OPTO43.C, OPTO44.C, OPTO45.C, OPTO46.C, OPTO47.C, OPTO48.C, OPTO5.C, OPTO6.C, OPTO7.C, OPTO8.C, OPTO9.C, Z1.A, Z10.A, Z11.A, Z12.A, Z13.A, Z14.A, Z15.A, Z16.A, Z17.A, Z18.A, Z19.A, Z2.A, Z20.A, Z21.A, Z22.A, Z23.A, Z24.A, Z25.A, Z26.A, Z27.A, Z28.A, Z29.A, Z3.A, Z30.A, Z31.A, Z32.A, Z33.A, Z34.A, Z35.A, Z36.A, Z37.A, Z38.A, Z39.A, Z4.A, Z40.A, Z41.A, Z42.A, Z43.A, Z44.A, Z45.A, Z46.A, Z47.A, Z48.A, Z5.A, Z6.A, Z7.A, Z8.A, Z9.A
- net GND: now also JP1.4, K22.S, Q9.E, RTC1.GND, U8.C
- net LED_PROSES: now also U3.IO25
- net LED_WARNING: now also U3.IO26
- net OUT+: now also D107.K, JP1.1, K21.1, R139.2
- net SCL: now also RTC1.SCL
- net SDA: now also RTC1.SDA
- net VCC: now also RTC1.VCC
